File: PCB/ESPPROG-Adapter.kicad_pcb (KiCad board)
At the start: 2 copper layers, 37.8 x 25.1 mm, 11 parts, among them J1 Conn_02x05_Odd_Even, J2 CONN ESP-PROG, J3 DebugHeader_Cortex-M_JTAG_10p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, J5 SOICBite connector UART Loopb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, J7 SOICBite IDC UART, J9 SOICBite IDC JTAG

Commit message: v1.5 TC2050 pinout change
Parts:
- J1: value Conn_02x05_Odd_Even -> Conn ESP-Prog JTAG
- J2: value CONN ESP-PROG -> Conn ESP-Prog UART
- J3: footprint jmux-footprints:TC-2050-IDC-SOCKET -> ESP-EZ-Debug:TC-2050-IDC-SOCKET
Routing:
- net /ESP_TMS: track 25.7 -> 34.2 mm, vias 0 -> 2
- net Net-(J3-~{RESET}): track 8.85 -> 3.11 mm
- net Earth: track 0.00 -> 4.14 mm, vias 8 -> 9
- net /ESP_TCK: track 31.7 -> 34.0 mm, vias 0 -> 1
- net /ESP_TDO: track 28.1 -> 29.6 mm, vias 2 -> 1
- net /ESP_TDI: track 38.7 -> 40.0 mm
Other:
- board text added: "0xjmux ${REVISION} 0324"
- board text removed: "0xjmux v1.4 02-2024"
