File: PCB/ESPPROG-Adapter.kicad_sch (KiCad schematic)
At the start: 12 parts, among them J1 Conn ESP-Prog JTAG, J2 Conn ESP-Prog UART, J3 DebugHeader_Cortex-M_JTAG_10p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, J5 SOICBite connector UART Loopb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, J7 SOICBite IDC UART, J8 SOICBite connector numbering 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, J9 SOICBite IDC JTAG

Commit message: v1.5 TC2050 pinout change
Parts:
- J3: footprint jmux-footprints:TC-2050-IDC-SOCKET -> ESP-EZ-Debug:TC-2050-IDC-SOCKET
Changed lines of the file:
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@@
 			)
 		)
-		(property "Footprint" "jmux-footprints:TC-2050-IDC-SOCKET"
+		(property "Footprint" "ESP-EZ-Debug:TC-2050-IDC-SOCKET"
 			(at 148.59 100.33 0)
 			(effects
@@
 			(at 160.02 102.87 0)
 			(effects
+				(font
+					(size 1.27 1.27)
+				)
+				(hide yes)
+			)
+		)
+		(property "Vendor" ""
+			(at 160.02 102.87 0)
+			(effects

Commit message: Clarification and new example added to SCH, links in library updated
* added link to hackaday article
* added clarification about CH_PD and GPIO2 to SCH
* Added example of ESP32 UART to SCH
* Added pinout table to README
* Updated example schematic
* replaced connector wiring example png with updated version
Other:
- note added: "Check out the ESP-EZ-Debug-KicadLib/ directory in the repo for symbols and footprints! (Link)"
- note added: "Connection Examples"
- note added: "ESP32 UART"
- note added: "ESP8266 UART"
- note added: "Original symbols for integrating SOICBite and TC2050 connector footprints into your ESP-based designs (jmux-kicad-things Link)"
- note added: "SOICBite JTAG"
- note added: "Tag-Connect ESP32 JTAG"
- note removed: "Below symbols for integrating SOICBite and TC2050 connector footprints into your ESP-based designs (jmux-kicad-things Link)"
